File: LED_7408_TASK/TASK_5.kicad_pcb (KiCad board)
At the start: 2 copper layers, 58.5 x 58.7 mm, 21 parts, among them J2 Conn_01x08_Pin, SW1 SW_DIP_x08

Commit message: KiCAD TASK
Parts:
- D1, D2, D3, D4, D5, D6, D7, D8, R1, R2, R3, R4, R5, R6, R7, R8: moved to F.Cu
- moved D6 1.42 mm to (144.6, 85.1)
- moved R6 1.41 mm to (141.9, 85.2)
- moved D7 0.91 mm to (144.3, 99.1)
- moved R7 0.91 mm to (141.6, 99.1)
- moved D8 0.85 mm to (144.3, 102.7)
- moved R8 0.84 mm to (141.5, 102.8)
- moved D4 0.76 mm to (144.1, 75.9)
- moved R4 0.75 mm to (141.4, 75.9)
- moved D5 0.75 mm to (143.8, 81.4)
- moved R5 0.75 mm to (141.1, 81.4)
- moved D3 0.58 mm to (144.1, 72.3)
- moved R3 0.58 mm to (141.3, 72.3)
- moved D2 0.54 mm to (144.0, 58.6)
- moved R2 0.54 mm to (141.3, 58.6)
- moved D1 0.50 mm to (144.0, 54.3)
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Routing:
- net GND: track 0.00 -> 139.2 mm, vias 0 -> 4
- net op6: track 3.53 -> 5.61 mm
- net op5: track 13.9 -> 12.3 mm
- net op3: track 7.93 -> 6.66 mm
- net op8: track 16.5 -> 15.5 mm
- net op7: track 7.29 -> 6.32 mm
- net op2: track 3.59 -> 4.48 mm
- net op4: track 16.8 -> 16.1 mm
